Commit message: Update hexapod tibia limits and standing pose

File: assets/robots/hexapod/urdf/hexapod.urdf (robot description, URDF)
Before this commit: robot hexapod, 19 links, 18 joints
Joints:
- joint BL_tibia_joint: limit lower=-2.443461 upper=0.000000 effort=10.0 velocity=10.0 -> lower=0.000000 upper=2.443461 effort=10.0 velocity=10.0
- joint BR_tibia_joint: limit lower=0.000000 upper=2.443461 effort=10.0 velocity=10.0 -> lower=-2.443461 upper=0.000000 effort=10.0 velocity=10.0
- joint FL_tibia_joint: limit lower=-2.443461 upper=0.000000 effort=10.0 velocity=10.0 -> lower=0.000000 upper=2.443461 effort=10.0 velocity=10.0
- joint FR_tibia_joint: limit lower=0.000000 upper=2.443461 effort=10.0 velocity=10.0 -> lower=-2.443461 upper=0.000000 effort=10.0 velocity=10.0
- joint ML_tibia_joint: limit lower=-2.443461 upper=0.000000 effort=10.0 velocity=10.0 -> lower=0.000000 upper=2.443461 effort=10.0 velocity=10.0
- joint MR_tibia_joint: limit lower=0.000000 upper=2.443461 effort=10.0 velocity=10.0 -> lower=-2.443461 upper=0.000000 effort=10.0 velocity=10.0

Commit message: Increase hexapod joint effort limits

File: assets/robots/hexapod/urdf/hexapod.urdf (robot description, URDF)
Before this commit: robot hexapod, 19 links, 18 joints
Joints:
- joint BL_coxa_joint: limit lower=-0.785398 upper=0.785398 effort=10.0 velocity=10.0 -> lower=-0.785398 upper=0.785398 effort=15.0 velocity=10.0
- joint BL_femur_joint: limit lower=-1.221730 upper=0.000000 effort=10.0 velocity=10.0 -> lower=-1.221730 upper=0.000000 effort=15.0 velocity=10.0
- joint BL_tibia_joint: limit lower=0.000000 upper=2.443461 effort=10.0 velocity=10.0 -> lower=0.000000 upper=2.443461 effort=15.0 velocity=10.0
- joint BR_coxa_joint: limit lower=-0.785398 upper=0.785398 effort=10.0 velocity=10.0 -> lower=-0.785398 upper=0.785398 effort=15.0 velocity=10.0
- joint BR_femur_joint: limit lower=0.000000 upper=1.221730 effort=10.0 velocity=10.0 -> lower=0.000000 upper=1.221730 effort=15.0 velocity=10.0
- joint BR_tibia_joint: limit lower=-2.443461 upper=0.000000 effort=10.0 velocity=10.0 -> lower=-2.443461 upper=0.000000 effort=15.0 velocity=10.0
- joint FL_coxa_joint: limit lower=-0.785398 upper=0.785398 effort=10.0 velocity=10.0 -> lower=-0.785398 upper=0.785398 effort=15.0 velocity=10.0
- joint FL_femur_joint: limit lower=-1.221730 upper=0.000000 effort=10.0 velocity=10.0 -> lower=-1.221730 upper=0.000000 effort=15.0 velocity=10.0
- joint FL_tibia_joint: limit lower=0.000000 upper=2.443461 effort=10.0 velocity=10.0 -> lower=0.000000 upper=2.443461 effort=15.0 velocity=10.0
- joint FR_coxa_joint: limit lower=-0.785398 upper=0.785398 effort=10.0 velocity=10.0 -> lower=-0.785398 upper=0.785398 effort=15.0 velocity=10.0
- joint FR_femur_joint: limit lower=0.000000 upper=1.221730 effort=10.0 velocity=10.0 -> lower=0.000000 upper=1.221730 effort=15.0 velocity=10.0
- joint FR_tibia_joint: limit lower=-2.443461 upper=0.000000 effort=10.0 velocity=10.0 -> lower=-2.443461 upper=0.000000 effort=15.0 velocity=10.0
- joint ML_coxa_joint: limit lower=-0.785398 upper=0.785398 effort=10.0 velocity=10.0 -> lower=-0.785398 upper=0.785398 effort=15.0 velocity=10.0
- joint ML_femur_joint: limit lower=-1.221730 upper=0.000000 effort=10.0 velocity=10.0 -> lower=-1.221730 upper=0.000000 effort=15.0 velocity=10.0
- joint ML_tibia_joint: limit lower=0.000000 upper=2.443461 effort=10.0 velocity=10.0 -> lower=0.000000 upper=2.443461 effort=15.0 velocity=10.0
- joint MR_coxa_joint: limit lower=-0.785398 upper=0.785398 effort=10.0 velocity=10.0 -> lower=-0.785398 upper=0.785398 effort=15.0 velocity=10.0
- joint MR_femur_joint: limit lower=0.000000 upper=1.221730 effort=10.0 velocity=10.0 -> lower=0.000000 upper=1.221730 effort=15.0 velocity=10.0
- joint MR_tibia_joint: limit lower=-2.443461 upper=0.000000 effort=10.0 velocity=10.0 -> lower=-2.443461 upper=0.000000 effort=15.0 velocity=10.0

Commit message: Increase hexapod torque limit to 50 Nm

File: assets/robots/hexapod/urdf/hexapod.urdf (robot description, URDF)
Before this commit: robot hexapod, 19 links, 18 joints
Joints:
- joint BL_coxa_joint: limit lower=-0.785398 upper=0.785398 effort=15.0 velocity=10.0 -> lower=-0.785398 upper=0.785398 effort=50.0 velocity=10.0
- joint BL_femur_joint: limit lower=-1.221730 upper=0.000000 effort=15.0 velocity=10.0 -> lower=-1.221730 upper=0.000000 effort=50.0 velocity=10.0
- joint BL_tibia_joint: limit lower=0.000000 upper=2.443461 effort=15.0 velocity=10.0 -> lower=0.000000 upper=2.443461 effort=50.0 velocity=10.0
- joint BR_coxa_joint: limit lower=-0.785398 upper=0.785398 effort=15.0 velocity=10.0 -> lower=-0.785398 upper=0.785398 effort=50.0 velocity=10.0
- joint BR_femur_joint: limit lower=0.000000 upper=1.221730 effort=15.0 velocity=10.0 -> lower=0.000000 upper=1.221730 effort=50.0 velocity=10.0
- joint BR_tibia_joint: limit lower=-2.443461 upper=0.000000 effort=15.0 velocity=10.0 -> lower=-2.443461 upper=0.000000 effort=50.0 velocity=10.0
- joint FL_coxa_joint: limit lower=-0.785398 upper=0.785398 effort=15.0 velocity=10.0 -> lower=-0.785398 upper=0.785398 effort=50.0 velocity=10.0
- joint FL_femur_joint: limit lower=-1.221730 upper=0.000000 effort=15.0 velocity=10.0 -> lower=-1.221730 upper=0.000000 effort=50.0 velocity=10.0
- joint FL_tibia_joint: limit lower=0.000000 upper=2.443461 effort=15.0 velocity=10.0 -> lower=0.000000 upper=2.443461 effort=50.0 velocity=10.0
- joint FR_coxa_joint: limit lower=-0.785398 upper=0.785398 effort=15.0 velocity=10.0 -> lower=-0.785398 upper=0.785398 effort=50.0 velocity=10.0
- joint FR_femur_joint: limit lower=0.000000 upper=1.221730 effort=15.0 velocity=10.0 -> lower=0.000000 upper=1.221730 effort=50.0 velocity=10.0
- joint FR_tibia_joint: limit lower=-2.443461 upper=0.000000 effort=15.0 velocity=10.0 -> lower=-2.443461 upper=0.000000 effort=50.0 velocity=10.0
- joint ML_coxa_joint: limit lower=-0.785398 upper=0.785398 effort=15.0 velocity=10.0 -> lower=-0.785398 upper=0.785398 effort=50.0 velocity=10.0
- joint ML_femur_joint: limit lower=-1.221730 upper=0.000000 effort=15.0 velocity=10.0 -> lower=-1.221730 upper=0.000000 effort=50.0 velocity=10.0
- joint ML_tibia_joint: limit lower=0.000000 upper=2.443461 effort=15.0 velocity=10.0 -> lower=0.000000 upper=2.443461 effort=50.0 velocity=10.0
- joint MR_coxa_joint: limit lower=-0.785398 upper=0.785398 effort=15.0 velocity=10.0 -> lower=-0.785398 upper=0.785398 effort=50.0 velocity=10.0
- joint MR_femur_joint: limit lower=0.000000 upper=1.221730 effort=15.0 velocity=10.0 -> lower=0.000000 upper=1.221730 effort=50.0 velocity=10.0
- joint MR_tibia_joint: limit lower=-2.443461 upper=0.000000 effort=15.0 velocity=10.0 -> lower=-2.443461 upper=0.000000 effort=50.0 velocity=10.0

Commit message: Use idealized hexapod actuator limits

File: assets/robots/hexapod/urdf/hexapod.urdf (robot description, URDF)
Before this commit: robot hexapod, 19 links, 18 joints
Joints:
- joint BL_coxa_joint: limit lower=-0.785398 upper=0.785398 effort=50.0 velocity=10.0 -> lower=-0.785398 upper=0.785398 effort=1000.0 velocity=100.0
- joint BL_femur_joint: limit lower=-1.221730 upper=0.000000 effort=50.0 velocity=10.0 -> lower=-1.221730 upper=0.000000 effort=1000.0 velocity=100.0
- joint BL_tibia_joint: limit lower=0.000000 upper=2.443461 effort=50.0 velocity=10.0 -> lower=0.000000 upper=2.443461 effort=1000.0 velocity=100.0
- joint BR_coxa_joint: limit lower=-0.785398 upper=0.785398 effort=50.0 velocity=10.0 -> lower=-0.785398 upper=0.785398 effort=1000.0 velocity=100.0
- joint BR_femur_joint: limit lower=0.000000 upper=1.221730 effort=50.0 velocity=10.0 -> lower=0.000000 upper=1.221730 effort=1000.0 velocity=100.0
- joint BR_tibia_joint: limit lower=-2.443461 upper=0.000000 effort=50.0 velocity=10.0 -> lower=-2.443461 upper=0.000000 effort=1000.0 velocity=100.0
- joint FL_coxa_joint: limit lower=-0.785398 upper=0.785398 effort=50.0 velocity=10.0 -> lower=-0.785398 upper=0.785398 effort=1000.0 velocity=100.0
- joint FL_femur_joint: limit lower=-1.221730 upper=0.000000 effort=50.0 velocity=10.0 -> lower=-1.221730 upper=0.000000 effort=1000.0 velocity=100.0
- joint FL_tibia_joint: limit lower=0.000000 upper=2.443461 effort=50.0 velocity=10.0 -> lower=0.000000 upper=2.443461 effort=1000.0 velocity=100.0
- joint FR_coxa_joint: limit lower=-0.785398 upper=0.785398 effort=50.0 velocity=10.0 -> lower=-0.785398 upper=0.785398 effort=1000.0 velocity=100.0
- joint FR_femur_joint: limit lower=0.000000 upper=1.221730 effort=50.0 velocity=10.0 -> lower=0.000000 upper=1.221730 effort=1000.0 velocity=100.0
- joint FR_tibia_joint: limit lower=-2.443461 upper=0.000000 effort=50.0 velocity=10.0 -> lower=-2.443461 upper=0.000000 effort=1000.0 velocity=100.0
- joint ML_coxa_joint: limit lower=-0.785398 upper=0.785398 effort=50.0 velocity=10.0 -> lower=-0.785398 upper=0.785398 effort=1000.0 velocity=100.0
- joint ML_femur_joint: limit lower=-1.221730 upper=0.000000 effort=50.0 velocity=10.0 -> lower=-1.221730 upper=0.000000 effort=1000.0 velocity=100.0
- joint ML_tibia_joint: limit lower=0.000000 upper=2.443461 effort=50.0 velocity=10.0 -> lower=0.000000 upper=2.443461 effort=1000.0 velocity=100.0
- joint MR_coxa_joint: limit lower=-0.785398 upper=0.785398 effort=50.0 velocity=10.0 -> lower=-0.785398 upper=0.785398 effort=1000.0 velocity=100.0
- joint MR_femur_joint: limit lower=0.000000 upper=1.221730 effort=50.0 velocity=10.0 -> lower=0.000000 upper=1.221730 effort=1000.0 velocity=100.0
- joint MR_tibia_joint: limit lower=-2.443461 upper=0.000000 effort=50.0 velocity=10.0 -> lower=-2.443461 upper=0.000000 effort=1000.0 velocity=100.0

Commit message: Add saturation-aware hexapod training signals

File: assets/robots/hexapod/urdf/hexapod.urdf (robot description, URDF)
Before this commit: robot hexapod, 19 links, 18 joints
Joints:
- joint BL_coxa_joint: limit lower=-0.785398 upper=0.785398 effort=1000.0 velocity=100.0 -> lower=-1.047198 upper=1.047198 effort=1000.0 velocity=100.0
- joint BR_coxa_joint: limit lower=-0.785398 upper=0.785398 effort=1000.0 velocity=100.0 -> lower=-1.047198 upper=1.047198 effort=1000.0 velocity=100.0
- joint FL_coxa_joint: limit lower=-0.785398 upper=0.785398 effort=1000.0 velocity=100.0 -> lower=-1.047198 upper=1.047198 effort=1000.0 velocity=100.0
- joint FR_coxa_joint: limit lower=-0.785398 upper=0.785398 effort=1000.0 velocity=100.0 -> lower=-1.047198 upper=1.047198 effort=1000.0 velocity=100.0
- joint ML_coxa_joint: limit lower=-0.785398 upper=0.785398 effort=1000.0 velocity=100.0 -> lower=-1.047198 upper=1.047198 effort=1000.0 velocity=100.0
- joint MR_coxa_joint: limit lower=-0.785398 upper=0.785398 effort=1000.0 velocity=100.0 -> lower=-1.047198 upper=1.047198 effort=1000.0 velocity=100.0
